File: preamplifier.kicad_sch (KiCad schematic)
At the start: 44 parts, among them SW1L1 SW_DIP_x04, SW1R1 SW_DIP_x04, U1 OPA2134, U2 OPA2134

Commit message: cosmetics
Other:
- note added: "Balance and Gain Control"
- note added: "First Amplification Stage Left Channel"
- note added: "First Amplification Stage Right Channel"
- note added: "Power Filtering"
- note added: "Second Amplification Stage Left Channel"
- note added: "Second Amplification Stage Right Channel"
- title: Preamplifier -> Audio Preamplifier
- moved on the sheet: C4, C5, C6, C7, C8, C9, RV1, RV2, U1A, U1B, U1C, U2A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
